Commit message: modifying the gripper description to add plate, fingers and porper simulation parameters (mass, inertia, ...)

File: wsg_50_simulation/urdf/wsg_50.urdf.xacro (robot description, xacro)
@@ -1,216 +1,423 @@
 <?xml version="1.0"?>
-<robot  xmlns:sensor="http://playerstage.sourceforge.net/gazebo/xmlschema/#sensor"
-	xmlns:controller="http://playerstage.sourceforge.net/gazebo/xmlschema/#controller"
-	xmlns:interface="http://playerstage.sourceforge.net/gazebo/xmlschema/#interface"
-        xmlns:xacro="http://ros.org/wiki/xacro"
-	name="wsg_50">
-<xacro:macro name="wsg_50_xacro" params="name parent *origin">
- <joint name="${name}_anterior_gripper_joint" type="fixed">
-    <insert_block name="origin"/>
-    <parent link="${parent}"/>
-    <child link="${name}_base_link"/>
- </joint>
-<!-- BASE LINK -->
- <link name="${name}_base_link">
-      <inertial>
-          <mass value="0.25" />
-          <origin xyz="0 0 0" />
-     	  <!--inertia ixx="1.0" ixy="0.0" ixz="0.0"
-               iyy="100.0" iyz="0.0"
-               izz="1.0" /-->
-      	  <inertia  ixx="1.0" ixy="0.0"  ixz="0.0"  iyy="1.0"  iyz="0.0"  izz="1.0" />
-      </inertial>
-      <visual>
-          <origin xyz="0.0 0 0" rpy="0 0 0" />
-          <geometry>
-             <mesh filename="package://wsg_50_simulation/meshes/WSG50_110.stl" scale="1 1 1"/>
-	     <!--box size="0.146 0.05 0.0735"/-->
-          </geometry>
-          <material name="grey">
-		<color rgba="0.5 0.5 0.5 1"/>
-      	  </material>
-      </visual>
-      <collision>
-          <origin xyz="0.0 0 0" rpy="0 0 0" />
-          <geometry>
-	     <!--box size="0.146 0.05 0.0735"/-->
-             <mesh filename="package://wsg_50_simulation/meshes/WSG50_110.stl" scale="1 1 1"/>
-         </geometry>
-     </collision>
-  </link>
-  <gazebo reference="${name}_base_link">
-    <material>Gazebo/Grey</material>
-    <turnGravityOff>false</turnGravityOff>
-  </gazebo>
-  <!-- GRIPPER LEFT -->
-  <joint name="${name}_base_joint_gripper_left" type="prismatic">
-     <limit lower="-0.055" upper="-0.0027" effort="1.0" velocity="1.0"/>
-     <origin xyz="0 0 0" rpy="0 0 0" />      <!--origin xyz="-0.0067 0 0.049" rpy="0 0 0" /-->
-     <parent link="${name}_base_link"/>
-     <child link="${name}_gripper_left" />
-     <dynamics friction="100" damping="100" />
-     <axis xyz="1 0 0"/>
-     <limit effort="100" velocity="100"/>
-  </joint>
-  <transmission name="${name}_base_trans_left" type="pr2_mechanism_model/SimpleTransmission">
-     <actuator name="${name}_base_motor_left" />
-     <joint name="${name}_base_joint_gripper_left" />
-     <mechanicalReduction>1</mechanicalReduction>
-     <motorTorqueConstant>1</motorTorqueConstant>
-  </transmission>
-  <link name="${name}_gripper_left">
-      <inertial>
-          <mass value="0.1" />
-          <origin xyz="0 0 0" />
-      <inertia ixx="1.0" ixy="0.0" ixz="0.0"
-               iyy="1.0" iyz="0.0"
-               izz="1.0" />
-      </inertial>
-      <visual>
-          <origin xyz="0.0 0 0" rpy="0 0 0" />
-          <geometry>
-             <mesh filename="package://wsg_50_simulation/meshes/GUIDE_WSG50_110.stl" scale="0.001 0.001 0.001"/>
-	     <!--box size="0.0175 0.03 0.024"/-->
-          </geometry>
-          <material name="black">
-		<color rgba="0 0 0 0"/>
-      	  </material>
-      </visual>
-      <collision>
-          <origin xyz="0 0 0" rpy="0 0 0" />
-          <geometry>
-	     <!--box size="0.0175 0.03 0.024"/-->
-             <mesh filename="package://wsg_50_simulation/meshes/GUIDE_WSG50_110.stl" scale="0.001 0.001 0.001"/>
-         </geometry>
-     </collision>
-     <contact_coefficients kd="1.0" kp="1000.0" mu="0"/>
-  </link>
-  <gazebo reference="${name}_gripper_left">
-    <material>Gazebo/Blue</material>
-    <turnGravityOff>false</turnGravityOff>
-  </gazebo>
-  <!-- LEFT FINGER -->
-  <joint name="${name}_guide_joint_finger_left" type="fixed">
-     <origin xyz="0 0 0.023" rpy="0 0 0" />
-     <parent link="${name}_gripper_left"/>
-     <child link="${name}_finger_left" />
-     <dynamics friction="100" damping="100" />
-     <axis xyz="1 0 0"/>
-     <limit effort="100" velocity="100"/>
-  </joint>
-  <link name="${name}_finger_left">
-      <inertial>
-          <mass value="0.1" />
-          <origin xyz="0 0 0" />
-      <inertia ixx="1.0" ixy="0.0" ixz="0.0"
-               iyy="1.0" iyz="0.0"
-               izz="1.0" />
-      </inertial>
-      <visual>
-          <origin xyz="0.0 0 0" rpy="0 0 0" />
-          <geometry>
-             <mesh filename="package://wsg_50_simulation/meshes/WSG-FMF.stl" scale="0.001 0.001 0.001"/>
-          </geometry>
-          <material name="black">
-		<color rgba="0 0 0 0"/>
-      	  </material>
-      </visual>
-      <collision>
-          <origin xyz="0 0 0" rpy="0 0 0" />
-          <geometry>
-             <mesh filename="package://wsg_50_simulation/meshes/WSG-FMF.stl" scale="0.001 0.001 0.001"/>
-         </geometry>
-     </collision>
-     <contact_coefficients kd="1.0" kp="1000.0" mu="0"/>
-  </link>
-  <gazebo reference="${name}_finger_left">
-    <material>Gazebo/Blue</material>
-    <turnGravityOff>false</turnGravityOff>
-  </gazebo>
-  <!-- GRIPPER RIGHT -->
-  <joint name="${name}_base_joint_gripper_right" type="prismatic">
-     <limit lower="0.0027" upper="0.055" effort="1.0" velocity="1.0"/>
-     <origin xyz="0 0 0" rpy="0 0 3.14159" />
-     <parent link="${name}_base_link"/>
-     <child link="${name}_gripper_right" />
-     <axis xyz="-1 0 0"/>
-     <dynamics friction="100" damping="100" />
-     <limit effort="100" velocity="100"/>
-  </joint>
-  <transmission name="${name}_base_trans_right" type="pr2_mechanism_model/SimpleTransmission">
-     <actuator name="${name}_base_motor_right" />
-     <joint name="${name}_base_joint_gripper_right" />
-     <mechanicalReduction>1</mechanicalReduction>
-     <motorTorqueConstant>1</motorTorqueConstant>
-  </transmission>
-    <link name="${name}_gripper_right">
-      <inertial>
-          <mass value="0.1" />
-          <origin xyz="0 0 0" />
-      <inertia ixx="1.0" ixy="0.0" ixz="0.0"
-               iyy="1.0" iyz="0.0"
-               izz="1.0" />
-      </inertial>
-      <visual>
-          <origin xyz="0.0 0 0" rpy="0 0 0" />
-          <geometry>
-             <mesh filename="package://wsg_50_simulation/meshes/GUIDE_WSG50_110.stl" scale="0.001 0.001 0.001"/>
-	     <!--box size="0.0175 0.03 0.024"/-->
-          </geometry>
-          <material name="black">
-		<color rgba="0 0 0 0"/>
-      	  </material>
-      </visual>
-      <collision>
-          <origin xyz="0 0 0" rpy="0 0 0" />
-          <geometry>
-	     <!--box size="0.0175 0.03 0.024"/-->
-             <mesh filename="package://wsg_50_simulation/meshes/GUIDE_WSG50_110.stl" scale="0.001 0.001 0.001"/>
-         </geometry>
-     </collision>
-     <contact_coefficients kd="1.0" kp="1000.0" mu="0"/>
-  </link>
-  <gazebo reference="gripper_right">
-    <material>Gazebo/White</material>
-    <turnGravityOff>false</turnGravityOff>
-  </gazebo>
-  <!-- RIGHT FINGER -->
-  <joint name="${name}_guide_joint_finger_right" type="fixed">
-     <origin xyz="0 0 0.023" rpy="0 0 0" />
-     <parent link="${name}_gripper_right"/>
-     <child link="${name}_finger_right" />
-     <dynamics friction="100" damping="100" />
-     <axis xyz="1 0 0"/>
-     <limit effort="100" velocity="100"/>
-  </joint>
-  <link name="${name}_finger_right">
-      <inertial>
-          <mass value="0.1" />
-          <origin xyz="0 0 0" />
-      <inertia ixx="1.0" ixy="0.0" ixz="0.0"
-               iyy="1.0" iyz="0.0"
-               izz="1.0" />
-      </inertial>
-      <visual>
-          <origin xyz="0.0 0 0" rpy="0 0 0" />
-          <geometry>
-             <mesh filename="package://wsg_50_simulation/meshes/WSG-FMF.stl" scale="0.001 0.001 0.001"/>
-          </geometry>
-          <material name="black">
-		<color rgba="0 0 0 0"/>
-      	  </material>
-      </visual>
-      <collision>
-          <origin xyz="0 0 0" rpy="0 0 0" />
-          <geometry>
-             <mesh filename="package://wsg_50_simulation/meshes/WSG-FMF.stl" scale="0.001 0.001 0.001"/>
-         </geometry>
-     </collision>
-     <contact_coefficients kd="1.0" kp="1000.0" mu="0"/>
-  </link>
-  <gazebo reference="${name}_finger_right">
-    <material>Gazebo/White</material>
-    <turnGravityOff>false</turnGravityOff>
-  </gazebo>
-</xacro:macro>
+<robot xmlns:sensor="http://playerstage.sourceforge.net/gazebo/xmlschema/#sensor"
+       xmlns:controller="http://playerstage.sourceforge.net/gazebo/xmlschema/#controller"
+       xmlns:interface="http://playerstage.sourceforge.net/gazebo/xmlschema/#interface"
+       xmlns:xacro="http://ros.org/wiki/xacro"
+       name="wsg_50">
+    <!-- finger_length: Length of finger from gripper base. (was 0.023) -->
+    <!-- finger_tip:    Offset of finger tip along fingers' motion direction.
+                        Use e.g. for single contact point tip on finger. (default 0) -->
+    <xacro:arg name="bubbles" default="False"/>
+    <xacro:macro name="wsg_50_xacro" params="name parent finger_length finger_tip hardware_interface *origin">
+        <joint name="${name}_plate_joint" type="fixed">
+            <xacro:insert_block name="origin"/>
+            <!-- <origin xyz="0 0 0" rpy="0 0 -1.5708"/> -->
+            <parent link="${parent}"/>
+            <child link="${name}_plate"/>
+        </joint>
+        <!-- GRIPPER PLATE -->
+        <link name="${name}_plate">
+          <inertial>
+            <mass value="0.0"/> <!-- This is not the true mass -->
+            <origin xyz="0 0 0"/>
+            <inertia ixx="1.0" ixy="0.0" ixz="0.0" iyy="1.0" iyz="0.0" izz="1.0"/> <!-- This are not the true inertia -->
+          </inertial>
+          <visual>
+            <origin rpy="0 0 0" xyz="0.0 0 0"/>
+            <geometry>
+              <mesh filename="package://med_description/meshes/wsg50/wsg50_plate.stl" scale="1 1 1"/>
+              <!--box size="0.146 0.05 0.0735"/-->
+            </geometry>
+            <material name="grey">
+              <color rgba="0.5 0.5 0.5 1"/>
+            </material>
+          </visual>
+          <collision>
+            <origin rpy="0 0 0" xyz="0.0 0 0"/>
+            <geometry>
+              <!--box size="0.146 0.05 0.0735"/-->
+              <mesh filename="package://med_description/meshes/wsg50/wsg50_plate.stl" scale="1 1 1"/>
+            </geometry>
+          </collision>
+        </link>
+        <gazebo reference="${name}_plate">
+          <material>Gazebo/Grey</material>
+          <turnGravityOff>false</turnGravityOff>
+        </gazebo>
+        <!-- GRIPPER -->
+        <joint name="${name}_anterior_gripper_joint" type="fixed">
+          <origin rpy="0 0 0" xyz="0 0 0.01"/>
+          <!-- <origin xyz="0 0 0" rpy="0 0 -1.5708"/> -->
+          <parent link="${name}_plate"/>
+          <child link="${name}_base_link"/>
+        </joint>
+        <!-- BASE LINK -->
+        <link name="${name}_base_link">
+            <inertial>
+                <mass value="1.48"/>
+                <origin xyz="0.00363 -0.00829 0.015"/>
+                <!--inertia ixx="1.0" ixy="0.0" ixz="0.0"
+                    iyy="100.0" iyz="0.0"
+                    izz="1.0" /-->
+                <inertia ixx="0.0" ixy="0.0" ixz="0.0" iyy="0.0" iyz="0.0" izz="0.0"/>
+            </inertial>
+            <visual>
+                <origin xyz="0.0 0 0" rpy="0 0 0"/>
+                <geometry>
+                    <mesh filename="package://med_description/meshes/wsg50/WSG50_110.stl" scale="1 1 1"/>
+                    <!--box size="0.146 0.05 0.0735"/-->
+                </geometry>
+                <material name="grey">
+                    <color rgba="0.5 0.5 0.5 1"/>
+                </material>
+            </visual>
+            <collision>
+                <origin xyz="0.0 0 0" rpy="0 0 0"/>
+                <geometry>
+                    <!--box size="0.146 0.05 0.0735"/-->
+                    <mesh filename="package://med_description/meshes/wsg50/WSG50_110.stl" scale="1 1 1"/>
+                </geometry>
+            </collision>
+        </link>
+        <gazebo reference="${name}_base_link">
+            <material>Gazebo/Grey</material>
+            <turnGravityOff>false</turnGravityOff>
+        </gazebo>
+        <joint name="${name}_center_joint" type="fixed">
+            <origin xyz="0 0 ${finger_length}" rpy="0 0 0"/>      <!--origin xyz="-0.0067 0 0.049" rpy="0 0 0" /-->
+            <parent link="${name}_base_link"/>
+            <child link="${name}_center"/>
+        </joint>
+        <link name="${name}_center">
+            <inertial>
+                <mass value="0"/>
+                <inertia ixx="0"  ixy="0"  ixz="0" iyy="0" iyz="0" izz="0" />
+            </inertial>
+        </link>
+        <!-- GRIPPER LEFT -->
+        <joint name="${name}_finger_left_joint" type="prismatic">
+            <limit lower="-0.055" upper="-0.03" effort="1.0" velocity="1.0"/>
+            <origin xyz="0 0 0" rpy="0 0 0"/>      <!--origin xyz="-0.0067 0 0.049" rpy="0 0 0" /-->
+            <parent link="${name}_base_link"/>
+            <child link="${name}_gripper_left"/>
+            <dynamics friction="100" damping="100"/>
+            <axis xyz="1 0 0"/>
+        </joint>
+        <transmission name="${name}_base_trans_left">
+            <type>transmission_interface/SimpleTransmission</type>
+            <actuator name="${name}_base_motor_left">
+                <mechanicalReduction>1</mechanicalReduction>
+            </actuator>
+            <joint name="${name}_finger_left_joint">
+                <hardwareInterface>${hardware_interface}</hardwareInterface>
+            </joint>
+        </transmission>
+        <link name="${name}_gripper_left">
+            <inertial>
+                <mass value="0.1"/>
+                <origin xyz="0 0 0"/>
+                <inertia ixx="1.0" ixy="0.0" ixz="0.0"
+                         iyy="1.0" iyz="0.0"
+                         izz="1.0"/>
+            </inertial>
+            <visual>
+                <origin xyz="0.0 0 0" rpy="0 0 0"/>
+                <geometry>
+                    <mesh filename="package://med_description/meshes/wsg50/GUIDE_WSG50_110.stl" scale="0.001 0.001 0.001"/>
+                    <!--box size="0.0175 0.03 0.024"/-->
+                </geometry>
+                <material name="black">
+                    <color rgba="0 0 0 1"/>
+                </material>
+            </visual>
+            <collision>
+                <origin xyz="0 0 0" rpy="0 0 0"/>
+                <geometry>
+                    <!--box size="0.0175 0.03 0.024"/-->
+                    <mesh filename="package://med_description/meshes/wsg50/GUIDE_WSG50_110.stl" scale="0.001 0.001 0.001"/>
+                </geometry>
+            </collision>
+            <contact_coefficients kd="1.0" kp="1000.0" mu="0"/>
+        </link>
+        <gazebo reference="${name}_gripper_left">
+            <material>Gazebo/Blue</material>
+            <turnGravityOff>false</turnGravityOff>
+        </gazebo>
+        <!-- LEFT FINGER -->
+        <xacro:if value="${$(arg bubbles) == False}">
+            <joint name="${name}_guide_joint_finger_left" type="fixed">
+                <origin xyz="${finger_tip} 0 ${finger_length}" rpy="0 0 0"/>
+                <parent link="${name}_gripper_left"/>
+                <child link="${name}_finger_left"/>
+                <dynamics friction="100" damping="100"/>
+                <axis xyz="1 0 0"/>
+                <limit effort="100" velocity="100"/>
+            </joint>
+            <link name="${name}_finger_left">
+                <inertial>
+                    <mass value="0.1"/>
+                    <origin xyz="0 0 0"/>
+                    <inertia ixx="1.0" ixy="0.0" ixz="0.0"
+                             iyy="1.0" iyz="0.0"
+                             izz="1.0"/>
+                </inertial>
+                <visual>
+                    <origin xyz="0.0 0 0" rpy="0 0 0"/>
+                    <geometry>
+                        <mesh filename="package://med_description/meshes/wsg50/WSG-FMF.stl" scale="0.001 0.001 0.001"/>
+                    </geometry>
+                    <material name="black">
+                        <color rgba="0 0 0 1"/>
+                    </material>
+                </visual>
+                <collision>
+                    <origin xyz="0 0 0" rpy="0 0 0"/>
+                    <geometry>
+                        <mesh filename="package://med_description/meshes/wsg50/WSG-FMF.stl" scale="0.001 0.001 0.001"/>
+                    </geometry>
+                </collision>
+                <contact_coefficients kd="1.0" kp="1000.0" mu="0"/>
+            </link>
+        </xacro:if>
+        <xacro:if value="$(arg bubbles)">
+            <!-- Bubbles -->
+            <joint name="${name}_guide_joint_finger_left" type="fixed">
+                <origin xyz="-0.009 0 .089" rpy="0 0 0"/>
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